Commit message: fix the 7dof urdf problem, and refactor the viz app

File: examples/models/ur5/ur5e+x.urdf (robot description, URDF)
Before this commit: robot ur5_with_x_axis, 15 links, 14 joints
Joints:
- joint external_axis_to_ur5_base_fixed: axis (none) -> 1.0 0.0 0.0; limit (none) -> lower=-1.5 upper=1.5 effort=1000 velocity=10; origin xyz=0.0 0.0 0.0 rpy=0.0 0.0 3.141592653589793 -> xyz=0.0 0.0 0.0 rpy=0.0 0.0 0.0; type fixed -> prismatic
- joint external_axis_x_joint: axis 1.0 0.0 0.0 -> (none); limit lower=-1.5 upper=1.5 effort=1000 velocity=10 -> (none); type prismatic -> fixed
